Commit message: Created core URDF

File: description/robot.urdf.xacro (robot description, xacro)
@@ -2,3 +2,4 @@
 <robot xmlns:xacro="http://www.ros.org/wiki/xacro"  name="robot">
   <xacro:include filename="robot_core.xacro" />
+  <xacro:include filename="gazebo_control.xacro" />
 </robot>

File: description/robot_core.xacro (robot description, xacro)
@@ -34,11 +34,14 @@
         <origin xyz="0.25 0 0.15" rpy="0 0 0"/>
         <geometry>
-            <cylinder length="0.3" radius="0.5" />
+            <cylinder length="0.2" radius="0.5" />
         </geometry>
     </collision>
-    <xacro:inertial_cylinder mass="0.5" length="0.3" radius="0.5">
+    <xacro:inertial_cylinder mass="0.5" length="0.2" radius="0.5">
         <origin xyz="0.25 0 0.15" rpy="0 0 0"/>
     </xacro:inertial_cylinder>
 </link>
+<gazebo reference="chassis">
+    <material>Gazebo/White</material>
+</gazebo>
 <!--LEFT WHEEL LINK-->
 <joint name="left_wheel_joint" type="continuous">
@@ -51,5 +54,5 @@
     <visual>
         <geometry>
-            <cylinder length="0.04" radius="0.05" />
+            <cylinder length="0.04" radius="0.165" />
         </geometry>
         <material name="blue"/>
@@ -57,11 +60,14 @@
     <collision>
         <geometry>
-            <cylinder length="0.04" radius="0.05" />
+            <cylinder length="0.04" radius="0.165" />
         </geometry>
     </collision>
-    <xacro:inertial_cylinder mass="0.1" length="0.04" radius="0.05">
+    <xacro:inertial_cylinder mass="0.1" length="0.04" radius="0.165">
         <origin xyz="0 0 0" rpy="0 0 0"/>
     </xacro:inertial_cylinder>
 </link>
+<gazebo reference="left_wheel">
+    <material>Gazebo/Blue</material>
+</gazebo>
 <!--RIGHT WHEEL LINK-->
 <joint name="right_wheel_joint" type="continuous">
@@ -74,5 +80,5 @@
     <visual>
         <geometry>
-            <cylinder length="0.04" radius="0.05" />
+            <cylinder length="0.04" radius="0.165" />
         </geometry>
         <material name="blue"/>
@@ -80,21 +86,24 @@
     <collision>
         <geometry>
-            <cylinder length="0.04" radius="0.05" />
+            <cylinder length="0.04" radius="0.165" />
         </geometry>
     </collision>
-    <xacro:inertial_cylinder mass="0.1" length="0.04" radius="0.05">
+    <xacro:inertial_cylinder mass="0.1" length="0.04" radius="0.165">
         <origin xyz="0 0 0" rpy="0 0 0"/>
     </xacro:inertial_cylinder>
 </link>
+<gazebo reference="right_wheel">
+    <material>Gazebo/Blue</material>
+</gazebo>
 <!-- CASTER WHEEL -->
 <joint name="caster_wheel_joint" type="fixed">
     <parent link="chassis"/>
     <child link="caster_wheel"/>
-    <origin xyz="0.4 0 0" rpy="0 0 0"/>
+    <origin xyz="0.5 0 0" rpy="0 0 0"/>
 </joint>
 <link name="caster_wheel">
     <visual>
         <geometry>
-            <sphere radius="0.05" />
+            <sphere radius="0.15" />
         </geometry>
         <material name="black"/>
@@ -102,11 +111,16 @@
     <collision>
         <geometry>
-            <sphere radius="0.05" />
+            <sphere radius="0.15" />
         </geometry>
         <material name="black"/>
     </collision>
-    <xacro:inertial_sphere mass="0.1" radius="0.05">
+    <xacro:inertial_sphere mass="0.1" radius="0.15">
         <origin xyz="0 0 0" rpy="0 0 0"/>
     </xacro:inertial_sphere>
 </link>
+<gazebo reference="castor_wheel">
+    <material>Gazebo/Black</material>
+    <mu1 value="0.002"/>
+    <mu2 value="0.002"/>
+</gazebo>
 </robot>

Commit message: Created core URDF

File: description/robot.urdf.xacro (robot description, xacro)
@@ -3,3 +3,4 @@
   <xacro:include filename="robot_core.xacro" />
   <xacro:include filename="gazebo_control.xacro" />
+  <xacro:include filename="lidar.xacro" />
 </robot>

File: description/robot_core.xacro (robot description, xacro)
@@ -13,4 +13,7 @@
     <material name="black">
         <color rgba="0 0 0 1"/>
+    </material>
+    <material name="red">
+        <color rgba="1 0 0 1"/>
     </material>
 <!--Base LINK -->
